Commit message: link ground to ur + fix ur position

File: mir250_ur16e_description/urdf/fixed_objects.urdf.xacro (robot description, xacro)
@@ -1,3 +1,4 @@
 <?xml version="1.0" ?>
+<robot xmlns:xacro="http://www.ros.org/wiki/xacro">
   <xacro:macro name="fixed_objects" params="
   tf_prefix
@@ -70,9 +71,14 @@
                 </collision>
         </link>
-        <joint name="ground_joint" type="fixed">
+	<joint name="ground_joint" type="fixed">
                 <parent link="${tf_prefix}world"/>
                 <child link="ground_plane"/>
                 <origin xyz="0 0 0" rpy="0 0 0"/>
-        </joint>                                                                                                                                                                                  <box size="0.35 0.55 0.55"/>                                                                                                                                                       </geometry>                                                                                                                                                                                <material name="very_red">                                                                                                                                                                         <color rgba="1 0 0 1"/>                                                                                                                                                            </material>                                                                                                                                                                        </collision>                                                                                                                                                                       </link>
+        </joint>
+        <joint name="ground_to_mir" type="fixed">
+                <parent link="ground_plane"/>
+                <child link="${tf_prefix}world"/>
+                <origin xyz="0 0 0" rpy="0 0 0"/>
+        </joint>
   </xacro:macro>
 </robot>

File: mir250_ur16e_description/urdf/ur_mir250_control.urdf.xacro (robot description, xacro)
@@ -6,5 +6,5 @@
   <xacro:include filename="$(find mir250_ur16e_description)/urdf/mir250_fixed.urdf.xacro"/>
   <xacro:include filename="$(find ur_description)/urdf/ur_macro.xacro"/>
-  <xacro:include filename="$(find mir250_ur16e_description)/urdf/fixed_objects.xacro"/>
+  <xacro:include filename="$(find mir250_ur16e_description)/urdf/fixed_objects.urdf.xacro"/>
   <!-- ros2 control include -->
   <xacro:include filename="$(find ur_robot_driver)/urdf/ur.ros2_control.xacro" />
@@ -76,5 +76,5 @@
     safety_k_position="$(arg safety_k_position)"
     >
-  <origin xyz="-0.155 0 -0.03" rpy="0 0 ${pi/2.0}" />          <!-- position robot in the world -->
+  <origin xyz="0.155 0 -0.03" rpy="0 0 -${pi/2.0}" />          <!-- position robot in the world -->
   </xacro:ur_robot>
   <!-- ros2 control instance -->

Commit message: adapt box and robot positions

File: mir250_ur16e_description/urdf/fixed_objects.urdf.xacro (robot description, xacro)
@@ -27,5 +27,5 @@
                 <parent link="platform"/>
                 <child link="control_box"/>
-                <origin xyz="-0.235 0 0.2575" rpy="0 0 0"/>
+                <origin xyz="-0.255 0 0.2575" rpy="0 0 0"/>
         </joint>
         <link name="platform">
@@ -71,9 +71,4 @@
                 </collision>
         </link>
-	<joint name="ground_joint" type="fixed">
-                <parent link="${tf_prefix}world"/>
-                <child link="ground_plane"/>
-                <origin xyz="0 0 0" rpy="0 0 0"/>
-        </joint>
         <joint name="ground_to_mir" type="fixed">
                 <parent link="ground_plane"/>

File: mir250_ur16e_description/urdf/ur_mir250_control.urdf.xacro (robot description, xacro)
@@ -76,5 +76,5 @@
     safety_k_position="$(arg safety_k_position)"
     >
-  <origin xyz="0.155 0 -0.03" rpy="0 0 -${pi/2.0}" />          <!-- position robot in the world -->
+  <origin xyz="0.22 0 -0.03" rpy="0 0 -${pi/2.0}" />          <!-- position robot in the world -->
   </xacro:ur_robot>
   <!-- ros2 control instance -->
